File: hagiwo-oscilloscope/hagiwo-oscilloscope.kicad_sch (KiCad schematic)
At the start: 4 parts

Commit message: further work on oscilloscope
Parts:
- added C3: 470pf, Capacitor_THT:C_Disc_D6.0mm_W2.5mm_P5.00mm, symbol Device:C
- added C4: 1uF, Capacitor_THT:C_Disc_D6.0mm_W2.5mm_P5.00mm, symbol Device:C
- added C5: 4.7 uF, Capacitor_THT:C_Disc_D6.0mm_W2.5mm_P5.00mm, symbol Device:C
- added C6, C7: 22 nF, Capacitor_THT:C_Disc_D6.0mm_W2.5mm_P5.00mm, symbol Device:C
- added D1, D2, D3, D4: D_Schottky, Diode_SMD:D_1210_3225Metric_Pad1.42x2.65mm_HandSolder, symbol Device:D_Schottky
- added J1: Encoder Header, Connector_JST:JST_XH_B5B-XH-A_1x05_P2.50mm_Vertical, symbol Connector:Conn_01x05_Female
- added J3: OLED Header, Connector_JST:JST_XH_B4B-XH-A_1x04_P2.50mm_Vertical, symbol Connector:Conn_01x04_Female
- added J4: Input Header, Connector_JST:JST_XH_B6B-XH-A_1x06_P2.50mm_Vertical, symbol Connector:Conn_01x06_Female
- added R1, R3: 47k O, Resistor_SMD:R_1210_3225Metric_Pad1.30x2.65mm_HandSolder, symbol Device:R_US
- added R2, R5: 10k O, Resistor_SMD:R_1210_3225Metric_Pad1.30x2.65mm_HandSolder, symbol Device:R_US
- added R4: 100k O, Resistor_SMD:R_1210_3225Metric_Pad1.30x2.65mm_HandSolder, symbol Device:R_US
- added R6, R7, R8: 1k O, Resistor_SMD:R_1210_3225Metric_Pad1.30x2.65mm_HandSolder, symbol Device:R_US
- added U1: Opamp_Dual, Package_DIP:DIP-8_W7.62mm_Socket, symbol Device:Opamp_Dual
- A1: renamed from A?; value Arduino_Nano_Every -> Nano
- C1, C2: renamed from C?; value 0.01pF -> 0.01uF; footprint (none) -> Capacitor_THT:C_Disc_D6.0mm_W2.5mm_P5.00mm
- gave numbers to parts that had none: 1
Connections:
- net +5V: now also D1.1 (K), D3.1 (K), J1.4 (Pin_4), J3.3 (Pin_3), U1.8 (V+)
- net EncoderCLK: now also J1.1 (Pin_1)
- net EncoderDT: now also J1.2 (Pin_2)
- net ExternalTrigger: now also D3.2 (A), D4.1 (K), R4.1, R7.2
- net GND: now also C3.2, C4.2, D2.2 (A), D4.2 (A), J1.5 (Pin_5), J3.4 (Pin_4), J4.6 (Pin_6), R4.2, U1.4 (V-); no longer A1.7 (D4)
- net LowPassInput: now also C6.1, C7.1
- net OLEDClock: now also J3.2 (Pin_2)
- net OLEDData: now also J3.1 (Pin_1)
- net OffsetVoltage: now also R3.2, R5.2, U1.1, U1.2 (-); no longer A1.12 (D9)
- net SignalIn: now also C3.1, C7.2, R8.1
- new net: D1.2 (A), D2.1 (K), R2.1, R3.1, U1.5 (+)
- new net: C6.2, R6.1, R8.2
- new net: C4.1, R1.1, U1.3 (+)
- new net ACInput: C5.2, J4.3 (Pin_3)
- new net DCInput: C5.1, J4.2 (Pin_2), R2.2
- new net EncoderSW: A1.7 (D4), J1.3 (Pin_3)
- new net OffsetOut: A1.12 (D9), R1.2
- new net PostGain: J4.5 (Pin_5), R6.2, U1.7
- new net PreGain: J4.4 (Pin_4), R5.1, U1.6 (-)
- new net TriggerJack: J4.1 (Pin_1), R7.1
Other:
- note added: "CORE"
- note added: "HEADERS"
- note added: "INPUT"
- note added: "OFFSET VOLTAGE"
- note added: "POWER"
- note added: "TRIGGER"
- moved on the sheet: A1, C1, C2, J2
