File: hagiwo-oscilloscope/hagiwo-oscilloscope-panel.kicad_pcb (KiCad board)
At the start: 2 copper layers, 139 x 110.2 mm, 26 parts, among them J1 Encoder Header, J2 10-Pin uZeus Power, J3 OLED Header, J4 Input Header, U1 Opamp_Dual

Commit message: defining panel pcb
Parts:
- removed REF**: Panel, oscfoot:Panel
Other:
- board size 139 x 110.2 mm -> 30.1 x 109.8 mm
Changed lines of the file:
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@@
-    )
-  )
-  (footprint "oscfoot:Panel" (layer "F.Cu")
-    (at 152.4 17.78)
-    (fp_text reference "REF**" (at 0 -0.5 unlocked) (layer "F.SilkS")
-      (effects (font (size 1 1) (thickness 0.15)))
-    )
-    (fp_text value "Panel" (at 0 1 unlocked) (layer "F.Fab")
-      (effects (font (size 1 1) (thickness 0.15)))
-    )
-    (fp_text user "${REFERENCE}" (at 0 2.5 unlocked) (layer "F.Fab")
-      (effects (font (size 1 1) (thickness 0.15)))
-    )
-    (fp_rect (start 0 0) (end 30.38 133.35) (layer "Edge.Cuts") (width 0.1) (fill none))
-    (fp_circle (center 27.77 3) (end 29.37 3) (layer "Edge.Cuts") (width 0.12) (fill none))
-    (fp_circle (center 7.45 130.35) (end 9.05 130.35) (layer "Edge.Cuts") (width 0.12) (fill none))
-    (fp_circle (center 27.77 130.35) (end 29.37 130.35) (layer "Edge.Cuts") (width 0.12) (fill none))
-    (fp_circle (center 7.45 3) (end 9.05 3) (layer "Edge.Cuts") (width 0.12) (fill none))
-    (group "" (id 06fe9e81-bb72-440d-ba0f-d15073a690ea)
-      (members
-        3950f8c9-6b09-48e0-8be8-6ce2c422ac1a
-        86cf6ff8-704a-4632-9b4d-a225e43f5054
-      )
-    )
-    (group "" (id 712af93f-80dd-4bbb-bc88-dd1aaae9070a)
-      (members
-        161e0b91-3cbe-4f94-bc6f-26d0f980024c
-        3c6a8808-4102-4851-aacf-c84c8cc5a7a9
-      )
     )
   )
@@
   (gr_circle (center 71.652 32.258) (end 73.152 32.258) (layer "Edge.Cuts") (width 0.1) (fill none))
   (gr_circle (center 71.628 138.43) (end 73.128 138.43) (layer "Edge.Cuts") (width 0.1) (fill none))
-  (gr_circle (center 180.856 139.192) (end 182.356 139.192) (layer "Edge.Cuts") (width 0.1) (fill none))
   (gr_rect (start 43.38 30.48) (end 73.46 140.24) (layer "Edge.Cuts") (width 0.1) (fill none))
-  (gr_circle (center 180.88 33.02) (end 182.38 33.02) (layer "Edge.Cuts") (width 0.1) (fill none))
-  (gr_circle (center 154.44 139.192) (end 155.94 139.192) (layer "Edge.Cuts") (width 0.1) (fill none))
-  (gr_circle (center 154.464 33.02) (end 155.964 33.02) (layer "Edge.Cuts") (width 0.1) (fill none))
   (gr_text "+12" (at 55.88 45.72) (layer "B.SilkS")
     (effects (font (size 1 1) (thickness 0.15)) (justify mirror))
@@
     (effects (font (size 1 1) (thickness 0.15)))
   )
-  (dimension (type aligned) (layer "Edge.Cuts")
-    (pts (xy 152.4 17.78) (xy 182.78 17.78))
-    (height -2.54)
-    (gr_text "30.3800 mm" (at 167.59 14.09) (layer "Edge.Cuts")
-      (effects (font (size 1 1) (thickness 0.15)))
-    )
-    (format (units 3) (units_format 1) (precision 4))
-    (style (thickness 0.1) (arrow_length 1.27) (text_position_mode 0) (extension_height 0.58642) (extension_offset 0.5) keep_text_aligned)
-  )
-  (dimension (type aligned) (layer "Edge.Cuts")
-    (pts (xy 182.78 17.78) (xy 182.78 151.13))
-    (height -5.18)
-    (gr_text "133.3500 mm" (at 186.81 84.455 90) (layer "Edge.Cuts")
-      (effects (font (size 1 1) (thickness 0.15)))
-    )
-    (format (units 3) (units_format 1) (precision 4))
-    (style (thickness 0.1) (arrow_length 1.27) (text_position_mode 0) (extension_height 0.58642) (extension_offset 0.5) keep_text_aligned)
-  )
   (dimension (type aligned) (layer "F.Fab")
